File: 【PBLED】Prayer Beads LED board2/【PBLED】Prayer Beads LED board2.sch (KiCad schematic (older format))
At the start: 175 parts, among them J1 PinSocket_1x01_Vertical, J10 PinSocket_1x01_Vertical, J11 PinSocket_1x01_Vertical, J12 PinSocket_1x01_Vertical, J13 PinSocket_1x01_Vertical, J14 PinSocket_1x01_Vertical, J15 PinSocket_1x01_Vertical, J16 PinSocket_1x01_Vertical, J17 PinSocket_1x01_Vertical, J18 PinSocket_1x01_Vertical, J19 PinSocket_1x01_Vertical, J2 PinSocket_1x01_Vertical, J20 PinSocket_1x01_Vertical, J21 PinSocket_1x01_Vertical, J22 PinSocket_1x01_Vertical, J23 PinSocket_1x01_Vertical, J24 PinSocket_1x01_Vertical, J25 PinSocket_1x01_Vertical, J26 PinSocket_1x01_Vertical, J27 PinSocket_1x01_Vertical, J28 PinSocket_1x01_Vertical, J29 PinSocket_1x01_Vertical, J3 PinSocket_1x01_Vertical, J30 PinSocket_1x01_Vertical, J31 PinSocket_1x01_Vertical, J32 PinSocket_1x08_Vertical, J33 PinSocket_1x01_Vertical, J34 PinSocket_1x01_Vertical, J35 PinSocket_1x01_Vertical, J36 PinSocket_1x01_Vertical, J37 PinSocket_1x01_Vertical, J38 PinSocket_1x01_Vertical, J39 PinSocket_1x01_Vertical, J4 PinSocket_1x01_Vertical, J40 PinSocket_1x01_Vertical, J41 PinSocket_1x01_Vertical, J42 PinSocket_1x01_Vertical, J43 PinSocket_1x01_Vertical, J44 PinSocket_1x01_Vertical, J45 PinSocket_1x01_Vertical, J46 PinSocket_1x01_Vertical, J47 PinSocket_1x01_Vertical, J48 PinSocket_1x01_Vertical, J49 PinSocket_1x01_Vertical, J5 PinSocket_1x01_Vertical, J50 PinSocket_1x01_Vertical, J51 PinSocket_1x01_Vertical, J52 PinSocket_1x01_Vertical, J53 PinSocket_1x01_Vertical, J54 PinSocket_1x01_Vertical, J55 PinSocket_1x01_Vertical, J56 PinSocket_1x01_Vertical, J57 PinSocket_1x01_Vertical, J58 PinSocket_1x01_Vertical, J59 PinSocket_1x01_Vertical, J6 PinSocket_1x01_Vertical, J60 PinSocket_1x01_Vertical, J61 PinSocket_1x01_Vertical, J62 PinSocket_1x01_Vertical, J63 PinSocket_1x01_Vertical, J64 PinSocket_1x01_Vertical, J65 PinSocket_1x01_Vertical, J7 PinSocket_1x01_Vertical, J8 PinSocket_1x01_Vertical, J9 PinSocket_1x01_Vertical, P1 Digital, P2 Analog, P3 CONN_01X01, P4 CONN_01X01, P5 CONN_01X01, P6 CONN_01X01, Q1 AO3400A, Q2 AO3400A, Q3 AO3400A, Q4 AO3400A, Q5 AO3400A, Q6 AO3400A, Q7 AO3400A, Q8 AO3400A, U1 LOGIC-74HC595D(SOIC16)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

Commit message: fix aaa
Parts:
- added U9: USB-C, Footprint-library:USB_C, symbol BAYASHI_Symbol-library:USB-C
- P1, P2: symbol 【PBLED】Prayer-Beads-LED-board2-rescue:Conn_01x15-Connector_Generic -> 【PBLED】Prayer-Beads-LED-board2-rescue:Conn_01x15-Connector_Generic-【PBLED】Prayer-Beads-LED-board2-rescue
- P3, P4, P5, P6: symbol 【PBLED】Prayer-Beads-LED-board2-rescue:Conn_01x01-Connector_Generic -> 【PBLED】Prayer-Beads-LED-board2-rescue:Conn_01x01-Connector_Generic-【PBLED】Prayer-Beads-LED-board2-rescue
- U1, U2, U3, U4, U5, U6, U7, U8: footprint SOIC16-1.27-10X3.9MM -> BAYASHI_Footprint-library:SOIC16-1.27-10X3.9MM; symbol Symbol-library:LOGIC-74HC595D(SOIC16) -> BAYASHI_Symbol-library:LOGIC-74HC595D(SOIC16)
Connections:
- net +5V: now also C11.2, C14.2, C17.2, C2.2, C20.2, C23.2, C5.2, C8.2, U1.10 (SCL), U1.16 (VCC), U2.10 (SCL), U2.16 (VCC), U3.10 (SCL), U3.16 (VCC), U4.10 (SCL), U4.16 (VCC), U5.10 (SCL), U5.16 (VCC), U6.10 (SCL), U6.16 (VCC), U7.10 (SCL), U7.16 (VCC), U8.10 (SCL), U8.16 (VCC), U9.A9 (VBUS), U9.B9 (VBUS)
- net GND: now also U9.A12 (GND), U9.B12 (GND)
- net +3V3: no longer names the net of P2.14 (Pin_14)
- net 13(SCK): no longer names the net of P2.15 (Pin_15)
- net AREF: no longer names the net of P2.13 (Pin_13)
- net Vin: no longer names the net of P2.1 (Pin_1)
- no-connect marks 20 -> 23
Other:
- moved on the sheet: J32, Q1, Q2, Q3, Q4, Q5, Q6, Q7, Q8
